Commit message: feat(3d): InMoov's wrists turn freely

File: public/models/inmoov/inmoov.urdf (robot description, URDF)
Before this commit: robot InMoov, 59 links, 58 joints
Joints:
- joint left_wrist_z_link_joint: limit lower=-1.5708 upper=1.5708 -> (none); type revolute -> continuous
- joint right_wrist_z_link_joint: limit lower=-1.5708 upper=1.5708 -> (none); type revolute -> continuous
